Commit message: feat: add HugWBC playback with wrist and hand control

File: source/robros_lab/robros_lab/assets/robots/robros/igris_c/from_urdf/urdf/igris_c_v2_wrist_hand_isaac.urdf (robot description, URDF)
Before this commit: robot IGRIS_C_WRIST_HAND, 56 links, 55 joints
Links:
- link Left_Hand: geometry collision box size=0.082 0.038 0.092; visual mesh filename=../meshes_v2/igris_c_end_effector/hand/l_palm.stl scale=0.01 0.01 0.01
- link Link_Wrist_Pitch_Left: geometry collision box size=0.028 0.020 0.030; visual mesh filename=../meshes_v2/igris_c_v2/l_wrist_connector.stl scale=0.01 0.01 0.01
- link Link_Wrist_Pitch_Right: geometry collision box size=0.028 0.020 0.030; visual mesh filename=../meshes_v2/igris_c_v2/r_wrist_connector.stl scale=0.01 0.01 0.01
- link Right_Hand: geometry collision box size=0.082 0.038 0.092; visual mesh filename=../meshes_v2/igris_c_end_effector/hand/r_palm.stl scale=0.01 0.01 0.01
- link l_thumb_distal: geometry collision cylinder length=0.030 radius=0.007; visual mesh filename=../meshes_v2/igris_c_end_effector/hand/l_thumb_distal.stl scale=0.01 0.01 0.01
- link l_thumb_middle: geometry collision cylinder length=0.034 radius=0.008; visual mesh filename=../meshes_v2/igris_c_end_effector/hand/l_thumb_middle.stl scale=0.01 0.01 0.01
- link l_thumb_proximal: geometry collision box size=0.035 0.018 0.018; visual mesh filename=../meshes_v2/igris_c_end_effector/hand/l_thumb_proximal.stl scale=0.01 0.01 0.01
- link r_thumb_distal: geometry collision cylinder length=0.030 radius=0.007; visual mesh filename=../meshes_v2/igris_c_end_effector/hand/r_thumb_distal.stl scale=0.01 0.01 0.01
- link r_thumb_middle: geometry collision cylinder length=0.034 radius=0.008; visual mesh filename=../meshes_v2/igris_c_end_effector/hand/r_thumb_middle.stl scale=0.01 0.01 0.01
- link r_thumb_proximal: geometry collision box size=0.035 0.018 0.018; visual mesh filename=../meshes_v2/igris_c_end_effector/hand/r_thumb_proximal.stl scale=0.01 0.01 0.01
